File: KiCAD-Project/JACC64-16K.kicad_sch (KiCad schematic)
At the start: 9 parts, among them SW1 SW_Push, U1 27C128

Commit message: Added PDF schematics
Other:
- note added: "VCC = +5V"
- company: (none) -> Oddsocks b5s4
